File: PCB/Motor_clock/DC-DC.sch (KiCad schematic (older format))
At the start: 9 parts

Commit message: Bug fix
Parts:
- L1: footprint Inductor_SMD:L_0603_1608Metric -> Inductor_SMD:L_Coilcraft_XAL5030
Changed lines of the file:
@@
 $Descr A4 11693 8268
 encoding utf-8
-Sheet 3 4
+Sheet 3 5
 Title ""
 Date ""
@@
 F 0 "L1" V 6685 3825 50  0000 C CNN
 F 1 "4.7uH" V 6594 3825 50  0000 C CNN
-F 2 "Inductor_SMD:L_0603_1608Metric" H 6500 3825 50  0001 C CNN
+F 2 "Inductor_SMD:L_Coilcraft_XAL5030" H 6500 3825 50  0001 C CNN
 F 3 "~" H 6500 3825 50  0001 C CNN
 	1    6500 3825
