File: PCB/Motor_clock/Motor_clock.sch (KiCad schematic (older format))
At the start: 27 parts

Commit message: commit
Parts:
- removed C?: 22u, symbol Device:C_Small
- removed C?: 0.1uF, symbol Device:C_Small
- removed C?: 47uF, symbol Device:C_Small
- removed D?: LED, symbol Device:LED
- removed L?: 4.7uH, symbol Device:L_Small
- removed R?: 10k, symbol Device:R_Small
- removed R?: 56.2k, symbol Device:R_Small
- removed R?: 1k, symbol Device:R_Small
- removed VR?: TPS561208DDCR, SOT95P280X110-6N, symbol TPS561208DDCR:TPS561208DDCR
- added J1: WS2812, Connector_JST:JST_PH_B3B-PH-K_1x03_P2.00mm_Vertical, symbol Connector:Conn_01x03_Female
- added R3, R4: 1k, Resistor_SMD:R_0603_1608Metric, symbol Device:R_Small
- BT1: renamed from BT?; footprint (none) -> CR1225:TE_796136-1
- C1, C2, C3, C4, C6: renamed from C?; footprint (none) -> Capacitor_SMD:C_0603_1608Metric
- C5: renamed from C?; value 4.7yF -> 4.7uF; footprint (none) -> Capacitor_SMD:C_0805_2012Metric
- J2: renamed from J?; footprint (none) -> DC_005:NINIGI_DC-005
- J3: renamed from J?; footprint (none) -> Connector_JST:JST_PH_S2B-PH-K_1x02_P2.00mm_Horizontal
- J4: renamed from J?; footprint (none) -> Connector_PinHeader_2.54mm:PinHeader_2x03_P2.54mm_Vertical
- R1, R2, R5: renamed from R?; footprint (none) -> Resistor_SMD:R_0603_1608Metric
- SW1, SW2: renamed from SW?; footprint (none) -> Button_Switch_SMD:SW_Push_1P1T_NO_6x6mm_H9.5mm
- Y1: renamed from Y?; footprint (none) -> Crystal:Crystal_SMD_3225-4Pin_3.2x2.5mm
- gave numbers to parts that had none: 2
Connections:
- net BAT_12V is gone; now on net 12V: J2.1, J3.1 (Pin_1)
- net +5V: now also J1.1 (Pin_1)
- net GND: now also J1.3 (Pin_3)
- net RESET: now also R1.2, SW2.2, U2.29 (~RESET~/PC6)
- net P2: now reaches U2.1 (PD3)
- net P5: now reaches U2.10 (PD6)
- net LED_DA: now reaches U2.11 (PD7)
- net LED_DA: now also J1.2 (Pin_2)
- net PDN: now reaches U2.12 (PB0)
- net P0: now reaches U2.13 (PB1)
- net DIR: now reaches U2.14 (PB2)
- net P3: now reaches U2.2 (PD4)
- net at U2.30 (PD0): now also R3.2
- net at U2.31 (PD1): now also R4.2
- net P1: now reaches U2.32 (PD2)
- net P4: now reaches U2.9 (PD5)
- new net RX: R4.1
- new net TX: R3.1
- no-connect marks 5 -> 9

Commit message: Bug fix
Parts:
- removed SW1: DS_reset, Button_Switch_SMD:SW_Push_1P1T_NO_6x6mm_H9.5mm, symbol Switch:SW_Push
- added BZ1: Buzzer, Buzzer:buzzer, symbol Device:Buzzer
- added C15: 100nF, Capacitor_SMD:C_0603_1608Metric, symbol Device:C_Small
- added D3: 1N5819, Diode_SMD:D_SMA, symbol Diode:1N5819
- added H1, H2, H3, H4: MountingHole, MountingHole:MountingHole_3.2mm_M3, symbol Mechanical:MountingHole
- added Q1: Q_NPN_BEC, Package_TO_SOT_SMD:SOT-23, symbol Device:Q_NPN_BEC
- added R9: 1k, Resistor_SMD:R_0603_1608Metric, symbol Device:R_Small
- J1: footprint Connector_JST:JST_PH_B3B-PH-K_1x03_P2.00mm_Vertical -> Connector_JST:JST_XH_S3B-XH-A-1_1x03_P2.50mm_Horizontal
Connections:
- net +5V: now also U1.4 (~RST)
- net 12V: now also BZ1.1 (-), C15.1, D3.1 (K)
- net GND: now also C15.2, Q1.2 (E)
- net PDN renamed Buzzer
- net Buzzer: now also R9.2
- new net: BZ1.2 (+), D3.2 (A), Q1.3 (C)
- new net: Q1.1 (B), R9.1
Other:
- note added: "Buzzer"
- note added: "Mounting_Hole\n"
Changed lines of the file:
@@
 $Descr A4 11693 8268
 encoding utf-8
-Sheet 1 4
+Sheet 1 5
 Title "Motor_clock"
 Date "2021-06-27"
@@
 	2350 4650 2450 4650
 $Comp
-L Switch:SW_Push SW1
-U 1 1 60DB61E2
-P 1150 4025
-F 0 "SW1" V 1196 3977 50  0000 R CNN
-F 1 "DS_reset" V 1105 3977 50  0000 R CNN
-F 2 "Button_Switch_SMD:SW_Push_1P1T_NO_6x6mm_H9.5mm" H 1150 4225 50  0001 C CNN
-F 3 "~" H 1150 4225 50  0001 C CNN
-	1    1150 4025
-	0    -1   -1   0
-$EndComp
-$Comp
 L power:GND #PWR0113
 U 1 1 60DB7699
@@
 	1650 3825 1150 3825
 Wire Wire Line
-	1150 4225 1150 4325
-Wire Wire Line
-	1150 4325 1325 4325
-Wire Wire Line
 	1325 4400 1325 4325
-Connection ~ 1325 4325
 Wire Wire Line
 	1325 4325 1450 4325
@@
 Text Notes 9175 2025 0    50   ~ 0
 POWER_Switch\n
-Text GLabel 4600 3525 2    50   Input ~ 0
-PDN
 Text GLabel 4600 3725 2    50   Input ~ 0
 DIR
@@
 F 0 "J1" H 8503 1301 50  0000 L CNN
 F 1 "WS2812" H 8503 1210 50  0000 L CNN
-F 2 "Connector_JST:JST_PH_B3B-PH-K_1x03_P2.00mm_Vertical" H 8475 1275 50  0001 C CNN
+F 2 "Connector_JST:JST_XH_S3B-XH-A-1_1x03_P2.50mm_Horizontal" H 8475 1275 50  0001 C CNN
 F 3 "~" H 8475 1275 50  0001 C CNN
 	1    8475 1275
@@
 LED_DA
 $Sheet
-S 3225 1250 1125 375
+S 2525 1250 1125 425
 U 60EF4BAF
 F0 "12V_5V" 50
@@
 U 1 1 60F29506
 P 4775 5225
-F 0 "R3" V 4579 5225 50  0000 C CNN
-F 1 "1k" V 4670 5225 50  0000 C CNN
+F 0 "R3" V 4700 5225 50  0000 C CNN
+F 1 "1k" V 4725 5350 50  0000 C CNN
 F 2 "Resistor_SMD:R_0603_1608Metric" H 4775 5225 50  0001 C CNN
 F 3 "~" H 4775 5225 50  0001 C CNN
@@
 U 1 1 60F2975F
 P 4775 5325
-F 0 "R4" V 4579 5325 50  0000 C CNN
-F 1 "1k" V 4670 5325 50  0000 C CNN
+F 0 "R4" V 4875 5400 50  0000 C CNN
+F 1 "1k" V 4725 5450 50  0000 C CNN
 F 2 "Resistor_SMD:R_0603_1608Metric" H 4775 5325 50  0001 C CNN
 F 3 "~" H 4775 5325 50  0001 C CNN
@@
 	4875 5325 4950 5325
 $Sheet
-S 4750 1250 900  200
+S 3900 1250 1000 425
 U 60F2F746
 F0 "USB2Serial" 50
@@
 Text GLabel 9950 2775 2    50   Input ~ 0
 12V
+$Sheet
+S 5100 1250 950  425
+U 60FD80B4
+F0 "TCA9548" 50
+F1 "TCA9548.sch" 50
+$EndSheet
+$Comp
+L Mechanical:MountingHole H1
+U 1 1 60FE3F7C
+P 9650 4350
+F 0 "H1" H 9750 4396 50  0000 L CNN
+F 1 "MountingHole" H 9750 4305 50  0000 L CNN
+F 2 "MountingHole:MountingHole_3.2mm_M3" H 9650 4350 50  0001 C CNN
+F 3 "~" H 9650 4350 50  0001 C CNN
+	1    9650 4350
+	1    0    0    -1
+$EndComp
+$Comp
+L Mechanical:MountingHole H2
+U 1 1 60FE463D
+P 9650 4625
+F 0 "H2" H 9750 4671 50  0000 L CNN
+F 1 "MountingHole" H 9750 4580 50  0000 L CNN
+F 2 "MountingHole:MountingHole_3.2mm_M3" H 9650 4625 50  0001 C CNN
+F 3 "~" H 9650 4625 50  0001 C CNN
+	1    9650 4625
+	1    0    0    -1
+$EndComp
+$Comp
+L Mechanical:MountingHole H3
+U 1 1 60FE4842
+P 9650 4900
+F 0 "H3" H 9750 4946 50  0000 L CNN
+F 1 "MountingHole" H 9750 4855 50  0000 L CNN
+F 2 "MountingHole:MountingHole_3.2mm_M3" H 9650 4900 50  0001 C CNN
+F 3 "~" H 9650 4900 50  0001 C CNN
+	1    9650 4900
+	1    0    0    -1
+$EndComp
+$Comp
+L Mechanical:MountingHole H4
+U 1 1 60FE4B1E
+P 9650 5175
+F 0 "H4" H 9750 5221 50  0000 L CNN
+F 1 "MountingHole" H 9750 5130 50  0000 L CNN
+F 2 "MountingHole:MountingHole_3.2mm_M3" H 9650 5175 50  0001 C CNN
+F 3 "~" H 9650 5175 50  0001 C CNN
+	1    9650 5175
+	1    0    0    -1
+$EndComp
+Wire Notes Line
+	9225 4150 10650 4150
+Wire Notes Line
+	10650 4150 10650 5400
+Wire Notes Line
+	10650 5400 9225 5400
+Wire Notes Line
+	9225 5400 9225 4150
+Text Notes 9225 4125 0    50   ~ 0
+Mounting_Hole\n
+$Comp
+L Device:Buzzer BZ1
+U 1 1 6101BB11
+P 8025 4550
+F 0 "BZ1" H 8177 4579 50  0000 L CNN
+F 1 "Buzzer" H 8177 4488 50  0000 L CNN
+F 2 "Buzzer:buzzer" V 8000 4650 50  0001 C CNN
+F 3 "~" V 8000 4650 50  0001 C CNN
+	1    8025 4550
+	1    0    0    -1
+$EndComp
+Text GLabel 4600 3525 2    50   Input ~ 0
+Buzzer
+Text GLabel 7300 5000 0    50   Input ~ 0
+Buzzer
+$Comp
+L power:GND #PWR03
+U 1 1 6101E943
+P 7800 5200
+F 0 "#PWR03" H 7800 4950 50  0001 C CNN
+F 1 "GND" H 7805 5027 50  0000 C CNN
+F 2 "" H 7800 5200 50  0001 C CNN
+F 3 "" H 7800 5200 50  0001 C CNN
+	1    7800 5200
+	1    0    0    -1
+$EndComp
+Text GLabel 7800 4350 1    50   Input ~ 0
+12V
+$Comp
+L Diode:1N5819 D3
+U 1 1 610FD42D
+P 7800 4600
+F 0 "D3" V 7754 4680 50  0000 L CNN
+F 1 "1N5819" V 7900 4450 50  0000 L CNN
+F 2 "Diode_SMD:D_SMA" H 7800 4425 50  0001 C CNN
+F 3 "http://www.vishay.com/docs/88525/1n5817.pdf" H 7800 4600 50  0001 C CNN
+	1    7800 4600
+	0    1    1    0
+$EndComp
+$Comp
+L Device:C_Small C15
+U 1 1 610FFA24
+P 7600 4550
+F 0 "C15" H 7350 4625 50  0000 L CNN
+F 1 "100nF" H 7275 4525 50  0000 L CNN
+F 2 "Capacitor_SMD:C_0603_1608Metric" H 7600 4550 50  0001 C CNN
+F 3 "~" H 7600 4550 50  0001 C CNN
+	1    7600 4550
+	1    0    0    -1
+$EndComp
+$Comp
+L Device:R_Small R9
+U 1 1 61104F68
+P 7400 5000
+F 0 "R9" V 7204 5000 50  0000 C CNN
+F 1 "1k" V 7295 5000 50  0000 C CNN
+F 2 "Resistor_SMD:R_0603_1608Metric" H 7400 5000 50  0001 C CNN
+F 3 "~" H 7400 5000 50  0001 C CNN
+	1    7400 5000
+	0    1    1    0
+$EndComp
+Wire Wire Line
+	7800 4350 7800 4450
+Wire Wire Line
+	7925 4450 7800 4450
+Connection ~ 7800 4450
+Wire Wire Line
+	7800 4450 7600 4450
+Wire Wire Line
+	7800 4800 7800 4775
+Wire Wire Line
+	7925 4650 7925 4775
+Wire Wire Line
+	7925 4775 7800 4775
+Connection ~ 7800 4775
+Wire Wire Line
+	7800 4775 7800 4750
+$Comp
+L power:GND #PWR05
+U 1 1 6110F7F2
+P 7600 4650
+F 0 "#PWR05" H 7600 4400 50  0001 C CNN
+F 1 "GND" H 7605 4477 50  0000 C CNN
+F 2 "" H 7600 4650 50  0001 C CNN
+F 3 "" H 7600 4650 50  0001 C CNN
+	1    7600 4650
+	1    0    0    -1
+$EndComp
+Wire Notes Line
+	8475 4125 8475 5500
+Wire Notes Line
+	8475 5500 6950 5500
+Wire Notes Line
+	6950 5500 6950 4125
+Wire Notes Line
+	6950 4125 8475 4125
+Text Notes 6925 4100 0    50   ~ 0
+Buzzer
+$Comp
+L power:+5V #PWR04
+U 1 1 6112775D
+P 1150 3825
+F 0 "#PWR04" H 1150 3675 50  0001 C CNN
+F 1 "+5V" H 1165 3998 50  0000 C CNN
+F 2 "" H 1150 3825 50  0001 C CNN
+F 3 "" H 1150 3825 50  0001 C CNN
+	1    1150 3825
+	1    0    0    -1
+$EndComp
+$Comp
+L Device:Q_NPN_BEC Q1
+U 1 1 6113DC4C
+P 7700 5000
+F 0 "Q1" H 7891 5046 50  0000 L CNN
+F 1 "Q_NPN_BEC" H 7891 4955 50  0000 L CNN
+F 2 "Package_TO_SOT_SMD:SOT-23" H 7900 5100 50  0001 C CNN
+F 3 "~" H 7700 5000 50  0001 C CNN
+	1    7700 5000
+	1    0    0    -1
+$EndComp
 $EndSCHEMATC
