File: PCB/Motor_clock/USB2Serial.sch (KiCad schematic (older format))
At the start: 12 parts, among them J11 USB_B_Micro, U9 CH340G, Y2 12Mhz

Commit message: Bug fix
Parts:
- removed D3, D4: LED, LED_SMD:LED_0603_1608Metric, symbol Device:LED
- removed R10, R9: 1k, Resistor_SMD:R_0603_1608Metric, symbol Device:R_Small
- added C14: 100nF, Capacitor_SMD:C_0603_1608Metric, symbol Device:C_Small
- J11: footprint Connector_USB:USB_Mini-B_AdamTech_MUSB-B5-S-VT-TSMT-1_SMD_Vertical -> USB:MicroXNJ
Connections:
- net RESET: now also C14.2; no longer U9.13 (~DTR)
- new net: C14.1, U9.13 (~DTR)
Changed lines of the file:
@@
 $Descr A4 11693 8268
 encoding utf-8
-Sheet 4 4
+Sheet 4 5
 Title ""
 Date ""
@@
 F 0 "J11" H 2307 4367 50  0000 C CNN
 F 1 "USB_B_Micro" H 2307 4276 50  0000 C CNN
-F 2 "Connector_USB:USB_Mini-B_AdamTech_MUSB-B5-S-VT-TSMT-1_SMD_Vertical" H 2400 3850 50  0001 C CNN
+F 2 "USB:MicroXNJ" H 2400 3850 50  0001 C CNN
 F 3 "~" H 2400 3850 50  0001 C CNN
 	1    2250 3900
@@
 RX
 $Comp
-L Device:R_Small R9
-U 1 1 60F3B0B8
-P 5475 3600
-F 0 "R9" H 5534 3646 50  0000 L CNN
-F 1 "1k" H 5534 3555 50  0000 L CNN
-F 2 "Resistor_SMD:R_0603_1608Metric" H 5475 3600 50  0001 C CNN
-F 3 "~" H 5475 3600 50  0001 C CNN
-	1    5475 3600
-	1    0    0    -1
-$EndComp
-$Comp
-L Device:LED D3
-U 1 1 60F3B67B
-P 5475 3850
-F 0 "D3" V 5514 3732 50  0000 R CNN
-F 1 "LED" V 5423 3732 50  0000 R CNN
-F 2 "LED_SMD:LED_0603_1608Metric" H 5475 3850 50  0001 C CNN
-F 3 "~" H 5475 3850 50  0001 C CNN
-	1    5475 3850
-	0    -1   -1   0
-$EndComp
-$Comp
-L Device:R_Small R10
-U 1 1 60F3CA69
-P 5725 3600
-F 0 "R10" H 5784 3646 50  0000 L CNN
-F 1 "1k" H 5784 3555 50  0000 L CNN
-F 2 "Resistor_SMD:R_0603_1608Metric" H 5725 3600 50  0001 C CNN
-F 3 "~" H 5725 3600 50  0001 C CNN
-	1    5725 3600
-	1    0    0    -1
-$EndComp
-$Comp
-L Device:LED D4
-U 1 1 60F3CD28
-P 5725 3850
-F 0 "D4" V 5764 3732 50  0000 R CNN
-F 1 "LED" V 5673 3732 50  0000 R CNN
-F 2 "LED_SMD:LED_0603_1608Metric" H 5725 3850 50  0001 C CNN
-F 3 "~" H 5725 3850 50  0001 C CNN
-	1    5725 3850
-	0    -1   -1   0
-$EndComp
-Wire Wire Line
-	5275 3250 5475 3250
-Wire Wire Line
-	5275 3350 5725 3350
-Wire Wire Line
-	5475 3500 5475 3250
-Connection ~ 5475 3250
-Wire Wire Line
-	5475 3250 5825 3250
-Wire Wire Line
-	5725 3350 5725 3500
-Connection ~ 5725 3350
-Wire Wire Line
-	5725 3350 5850 3350
-$Comp
-L power:GND #PWR0131
-U 1 1 60F3E7D5
-P 5625 4125
-F 0 "#PWR0131" H 5625 3875 50  0001 C CNN
-F 1 "GND" H 5630 3952 50  0000 C CNN
-F 2 "" H 5625 4125 50  0001 C CNN
-F 3 "" H 5625 4125 50  0001 C CNN
-	1    5625 4125
-	1    0    0    -1
-$EndComp
-Wire Wire Line
-	5475 4000 5475 4125
-Wire Wire Line
-	5475 4125 5625 4125
-Wire Wire Line
-	5725 4125 5725 4000
-Connection ~ 5625 4125
-Wire Wire Line
-	5625 4125 5725 4125
-$Comp
 L Device:C_Small C12
 U 1 1 60F3FA49
@@
 Wire Wire Line
 	5325 3950 5325 4250
-Text GLabel 5325 4250 3    50   Input ~ 0
+Text GLabel 5325 4450 3    50   Input ~ 0
 RESET
 $Comp
@@
 	4875 3025 5050 3025
 Connection ~ 4875 3025
+$Comp
+L Device:C_Small C14
+U 1 1 60FCECB7
+P 5325 4350
+F 0 "C14" H 5417 4396 50  0000 L CNN
+F 1 "100nF" H 5417 4305 50  0000 L CNN
+F 2 "Capacitor_SMD:C_0603_1608Metric" H 5325 4350 50  0001 C CNN
+F 3 "~" H 5325 4350 50  0001 C CNN
+	1    5325 4350
+	1    0    0    -1
+$EndComp
+Wire Wire Line
+	5275 3250 5825 3250
+Wire Wire Line
+	5275 3350 5850 3350
 $EndSCHEMATC
